Commit message: modify universal robot

File: ur_description/urdf/inc/ur_macro.xacro (robot description, xacro)
@@ -44,4 +44,6 @@
   <xacro:include filename="$(find ur_description)/urdf/inc/ur_transmissions.xacro" />
   <xacro:include filename="$(find ur_description)/urdf/inc/ur_common.xacro" />
+  <xacro:include filename="$(find dh_robotics_ag95_description)/urdf/dh_robotics_ag95_gripper.urdf.xacro"/>
+  <xacro:include filename="$(find realsense2_description)/urdf/_d435.urdf.xacro"/>
   <xacro:macro name="ur_robot" params="
     prefix
@@ -64,5 +66,5 @@
     <xacro:ur_arm_transmission prefix="${prefix}" hw_interface="${transmission_hw_interface}" />
     <!-- links: main serial chain -->
-    <link name="${prefix}base_link"/>
+    <!--link name="${prefix}base_link"/-->
     <link name="${prefix}base_link_inertia">
       <visual>
@@ -215,5 +217,5 @@
            link/frame) to introduce the necessary rotation over Z (of pi rad).
       -->
-      <origin xyz="0 0 0" rpy="0 0 ${pi}" />
+      <origin xyz="0.13 0 0.421" rpy="0 0 ${pi/2}" />
     </joint>
     <joint name="${prefix}shoulder_pan_joint" type="revolute">
@@ -291,5 +293,5 @@
     <!-- ROS-Industrial 'base' frame: base_link to UR 'Base' Coordinates transform -->
     <link name="${prefix}base"/>
-    <joint name="${prefix}base_link-base_fixed_joint" type="fixed">
+   <joint name="${prefix}base_link-base_fixed_joint" type="fixed">
       <!-- Note the rotation over Z of pi radians: as base_link is REP-103
            aligned (ie: has X+ forward, Y+ left and Z+ up), this is needed
@@ -317,3 +319,9 @@
     </joint>
   </xacro:macro>
+  <xacro:dh_robotics_ag95_gripper prefix="" parent="wrist_3_link" >
+        <origin xyz="0 0 0.02" rpy="0 0 0"/>
+  </xacro:dh_robotics_ag95_gripper>
+  <xacro:sensor_d435 parent="wrist_3_link" name="sensor_d435" >
+        <origin xyz="0 0.1 0.03" rpy="${-pi/2} ${-pi/2} 0"/>
+  </xacro:sensor_d435>
 </robot>

Commit message: gazebo

File: ur_description/urdf/inc/ur_macro.xacro (robot description, xacro)
@@ -44,6 +44,4 @@
   <xacro:include filename="$(find ur_description)/urdf/inc/ur_transmissions.xacro" />
   <xacro:include filename="$(find ur_description)/urdf/inc/ur_common.xacro" />
-  <xacro:include filename="$(find dh_robotics_ag95_description)/urdf/dh_robotics_ag95_gripper.urdf.xacro"/>
-  <xacro:include filename="$(find realsense2_description)/urdf/_d435.urdf.xacro"/>
   <xacro:macro name="ur_robot" params="
     prefix
@@ -217,5 +215,5 @@
            link/frame) to introduce the necessary rotation over Z (of pi rad).
       -->
-      <origin xyz="0.13 0 0.421" rpy="0 0 ${pi/2}" />
+      <origin xyz="0.14 0 0.41" rpy="0 0 ${pi/2}" />
     </joint>
     <joint name="${prefix}shoulder_pan_joint" type="revolute">
@@ -293,5 +291,5 @@
     <!-- ROS-Industrial 'base' frame: base_link to UR 'Base' Coordinates transform -->
     <link name="${prefix}base"/>
-   <joint name="${prefix}base_link-base_fixed_joint" type="fixed">
+    <joint name="${prefix}base_link-base_fixed_joint" type="fixed">
       <!-- Note the rotation over Z of pi radians: as base_link is REP-103
            aligned (ie: has X+ forward, Y+ left and Z+ up), this is needed
@@ -319,9 +317,3 @@
     </joint>
   </xacro:macro>
-  <xacro:dh_robotics_ag95_gripper prefix="" parent="wrist_3_link" >
-        <origin xyz="0 0 0.02" rpy="0 0 0"/>
-  </xacro:dh_robotics_ag95_gripper>
-  <xacro:sensor_d435 parent="wrist_3_link" name="sensor_d435" >
-        <origin xyz="0 0.1 0.03" rpy="${-pi/2} ${-pi/2} 0"/>
-  </xacro:sensor_d435>
 </robot>
