Commit message: change for first lecture

File: tracer_ros/tracer_description/urdf/tracer_v1.xacro (robot description, xacro)
@@ -144,3 +144,7 @@
     <!-- Gazebo definitions  -->
     <xacro:include filename="$(find tracer_description)/urdf/tracer.gazebo" />
+    <xacro:include filename="$(find velodyne_description)/urdf/VLP-16.urdf.xacro"/>
+    <xacro:VLP-16 parent="base_link" name="velodyne" topic="/velodyne_points" hz="10" samples="440" gpu="false">
+        <origin xyz="0.3 0 0.15" rpy="0 0 0" />
+    </xacro:VLP-16>
 </robot>
